File: orange_lamp.kicad_pcb (KiCad board)
At the start: 2 copper layers, 65 x 8 mm, 13 parts, among them J1 POWER, J2 LEDIN, J3 LEDOUT, U1 LM317_TO-252

Commit message: Final PCB.
Parts:
- moved JP1 5.11 mm to (143.0, 54.6)
Other:
- board text added: "+"
- board text added: "-"
- board text added: "GND"
- board text added: "LED IN"
- board text added: "LED OUT"
- board text added: "Orange LED driver v1 Jethro, 2022"
- board text added: "VCC IN"
- board text added: "Vin: 9-36V, Iout: 36mA"
Changed lines of the file:
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@@
     (property "Sheetname" "")
     (attr smd)
-    (fp_text reference "R1" (at 0 -1.65 90) (layer "F.SilkS")
+    (fp_text reference "R1" (at 1.4569 -4.79 90) (layer "F.SilkS")
       (effects (font (size 1 1) (thickness 0.15)))
     )
@@
     (property "Sheetname" "")
     (attr smd)
-    (fp_text reference "D1" (at 0 -2.5 90) (layer "F.SilkS")
+    (fp_text reference "D1" (at 3.1 1.9 90) (layer "F.SilkS")
       (effects (font (size 1 1) (thickness 0.15)))
     )
@@
     (property "Sheetname" "")
     (attr smd)
-    (fp_text reference "C2" (at 0 -1.85 90) (layer "F.SilkS")
+    (fp_text reference "C2" (at 0.1806 2.6056 90) (layer "F.SilkS")
       (effects (font (size 1 1) (thickness 0.15)))
     )
@@
     (property "Sheetname" "")
     (attr smd)
-    (fp_text reference "C1" (at 0 -1.43 90) (layer "F.SilkS")
+    (fp_text reference "C1" (at -0.225 -4.7 90) (layer "F.SilkS")
       (effects (font (size 1 1) (thickness 0.15)))
     )
@@
     (property "Sheetname" "")
     (attr through_hole)
-    (fp_text reference "J2" (at -3.7573 -6.2536 90) (layer "F.SilkS")
+    (fp_text reference "J2" (at 1.17 3.9 90) (layer "F.SilkS")
       (effects (font (size 1 1) (thickness 0.15)))
     )
@@
     (property "Sheetname" "")
     (attr smd)
-    (fp_text reference "U1" (at 0 -4.5) (layer "F.SilkS")
+    (fp_text reference "U1" (at 6.3696 -2.7 90) (layer "F.SilkS")
       (effects (font (size 1 1) (thickness 0.15)))
     )
@@
     (property "Sheetname" "")
     (attr through_hole)
-    (fp_text reference "J1" (at 1.27 -4.12 90) (layer "F.SilkS")
+    (fp_text reference "J1" (at 4.57 -2.22 180) (layer "F.SilkS")
       (effects (font (size 1 1) (thickness 0.15)))
     )
@@
     (property "Sheetname" "")
     (attr through_hole)
-    (fp_text reference "J3" (at 1.27 -4.12 90) (layer "F.SilkS")
+    (fp_text reference "J3" (at 3.37 -3.7 90) (layer "F.SilkS")
       (effects (font (size 1 1) (thickness 0.15)))
     )
@@
   )
   (footprint "Jumper:SolderJumper-2_P1.3mm_Open_TrianglePad1.0x1.5mm" (layer "B.Cu")
-    (at 137.8892 54.5878 -90)
+    (at 143 54.6 -90)
     (descr "SMD Solder Jumper, 1x1.5mm Triangular Pads, 0.3mm gap, open")
     (tags "solder jumper open")
@@
         (gr_poly (pts
             (xy 1 0)
+            (xy 0.5 0.75)
+            (xy -0.5 0.75)
+            (xy -0.5 -0.75)
             (xy 0.5 -0.75)
-            (xy -0.5 -0.75)
-            (xy -0.5 0.75)
-            (xy 0.5 0.75)
           ) (width 0) (fill yes))
       ))
@@
       (primitives
         (gr_poly (pts
+            (xy 0.5 0.75)
+            (xy -0.65 0.75)
+            (xy -0.15 0)
+            (xy -0.65 -0.75)
             (xy 0.5 -0.75)
-            (xy -0.65 -0.75)
-            (xy -0.15 0)
-            (xy -0.65 0.75)
-            (xy 0.5 0.75)
           ) (width 0) (fill yes))
       ))
   )
+  (gr_line (start 108.8 57.8) (end 108.6 57.6) (layer "F.SilkS") (width 0.15))
+  (gr_line (start 112.4 52.4) (end 109.6 52.4) (layer "F.SilkS") (width 0.15))
+  (gr_line (start 112.6 57.8) (end 109.6 57.8) (layer "F.SilkS") (width 0.15))
+  (gr_line (start 109.6 57.8) (end 108.8 57.8) (layer "F.SilkS") (width 0.15))
   (gr_line (start 144.5 50.5) (end 79.5 50.5) (layer "Edge.Cuts") (width 0.1))
   (gr_line (start 79.5 50.5) (end 79.5 58.5) (layer "Edge.Cuts") (width 0.1))
   (gr_line (start 144.5 58.5) (end 144.5 50.5) (layer "Edge.Cuts") (width 0.1))
   (gr_line (start 79.5 58.5) (end 144.5 58.5) (layer "Edge.Cuts") (width 0.1))
+  (gr_text "GND" (at 85.4 52.8 90) (layer "B.SilkS")
+    (effects (font (size 1 1) (thickness 0.15)) (justify mirror))
+  )
+  (gr_text "LED\nIN" (at 114.4 56.2 90) (layer "B.SilkS")
+    (effects (font (size 1 1) (thickness 0.15)) (justify mirror))
+  )
+  (gr_text "GND" (at 115.2 52.6 90) (layer "B.SilkS")
+    (effects (font (size 1 1) (thickness 0.15)) (justify mirror))
+  )
+  (gr_text "Vin: 9-36V, Iout: 36mA" (at 98.4 55.8) (layer "B.SilkS")
+    (effects (font (size 1 1) (thickness 0.15)) (justify mirror))
+  )
+  (gr_text "VCC\nIN" (at 86.2 56.4 90) (layer "B.SilkS")
+    (effects (font (size 1 1) (thickness 0.15)) (justify mirror))
+  )
+  (gr_text "Orange LED driver v1\nJethro, 2022" (at 128.4 54) (layer "B.SilkS")
+    (effects (font (size 1 1) (thickness 0.15)) (justify mirror))
+  )
+  (gr_text "GND" (at 138.2 52.6 90) (layer "B.SilkS")
+    (effects (font (size 1 1) (thickness 0.15)) (justify mirror))
+  )
+  (gr_text "LED\nOUT" (at 137.4 56.2 90) (layer "B.SilkS")
+    (effects (font (size 1 1) (thickness 0.15)) (justify mirror))
+  )
+  (gr_text "+\n" (at 141.2 57.8) (layer "F.SilkS")
+    (effects (font (size 1 1) (thickness 0.15)))
+  )
+  (gr_text "-" (at 117.4 51.2) (layer "F.SilkS")
+    (effects (font (size 1 1) (thickness 0.15)))
+  )
+  (gr_text "+" (at 117.4 57.8) (layer "F.SilkS")
+    (effects (font (size 1 1) (thickness 0.15)))
+  )
+  (gr_text "+" (at 83 57.8) (layer "F.SilkS")
+    (effects (font (size 1 1) (thickness 0.15)))
+  )
+  (gr_text "-" (at 140.4 51.2) (layer "F.SilkS")
+    (effects (font (size 1 1) (thickness 0.15)))
+  )
+  (gr_text "-" (at 83 51.2) (layer "F.SilkS")
+    (effects (font (size 1 1) (thickness 0.15)))
+  )
   (segment (start 92.5492 52.21) (end 92.2592 52.5) (width 1) (layer "F.Cu") (net 1))
   (segment (start 108.5 51.45) (end 106.3396 51.45) (width 1) (layer "F.Cu") (net 1))
@@
   (segment (start 137.75 53) (end 134.608 53) (width 1) (layer "F.Cu") (net 12))
   (segment (start 140.5 55.75) (end 137.75 53) (width 1) (layer "F.Cu") (net 12))
-  (segment (start 137.8892 55.3128) (end 140.0428 55.3128) (width 0.5) (layer "B.Cu") (net 12))
-  (segment (start 140.0428 55.3128) (end 140.5 55.77) (width 0.5) (layer "B.Cu") (net 12))
+  (segment (start 140.5 55.77) (end 140.82048 55.44952) (width 0.75) (layer "B.Cu") (net 12))
+  (segment (start 140.82048 55.44952) (end 143 55.44952) (width 0.75) (layer "B.Cu") (net 12))
   (zone (net 13) (net_name "unconnected-(D5-Pad2)") (layer "F.Cu") (hatch edge 0.508)
     (priority 1)
